Commit message: Revert "new"
This reverts commit 157a2a88b99d6f00a54721e31e290ad2fbe3db87.

File: arpg/ros_ws/src/simulation/racer_description/urdf/racer.xacro (robot description, xacro)
@@ -14,5 +14,4 @@
   <xacro:property name="bodySizeH" value="0.1"/>
   <xacro:property name="bodyMass" value="3.5"/>
-  <xacro:arg name="car_highlighting" default="false"/>
   <link name="base_link" />
   <joint name="base_link_joint" type="fixed">
@@ -41,9 +40,4 @@
     </visual>
   </link>
-  <xacro:if value="$(arg car_highlighting)">
-    <gazebo reference="chassis">
-      <material>Gazebo/GreenGlow</material>
-    </gazebo>
-  </xacro:if>
   <!--  Wheels  -->
   <wheel fb="front" lr="left" parent="left_steering" translateX="1" translateY="1" left="1" OffsetJointX= "${base_x_sphere_origin_to_wheel_origin}" OffsetJointY= "${base_y_sphere_origin_to_wheel_origin}" OffsetJointZ= "${base_z_sphere_origin_to_wheel_origin}" OffsetY="0.02" />
